Commit message: adding mocap link to table (pick works in sim)

File: agimus_demo_10_tiago_pro_bar_manip/urdf/macro/table_macro.urdf.xacro (robot description, xacro)
@@ -37,4 +37,10 @@
       </collision>
     </link>
+    <link name="mocap_table"/>
+    <joint name="mocap_to_table" type="fixed">
+      <parent link="table_link"/>
+      <child link="mocap_table"/>
+      <origin xyz="0.7 -0.7 0" rpy="0 0 1.57"/>
+    </joint>
   </xacro:macro>
 </robot>
