Commit message: Add sim option into launch + cancel exec

File: agimus_demo_10_tiago_pro_bar_manip/urdf/environment.urdf.xacro (robot description, xacro)
@@ -17,5 +17,5 @@
     <parent link="world"/>
     <child link="table_link"/>
-    <origin xyz="2.9 0 0.74" rpy="0 0 3.14"/>
+    <origin xyz="2.3 0 0.74" rpy="0 0 3.14"/>
   </joint>
   <xacro:bordered_plate name="plate">
@@ -25,5 +25,5 @@
     <parent link="table_link"/>
     <child link="plate_base_link"/>
-    <origin xyz="0 0 0.015" rpy="0 0 0"/>
+    <origin xyz="-0.2 0 0" rpy="0 0 0"/>
   </joint>
   <xacro:support_bar spacing="0.95"/>
@@ -31,5 +31,5 @@
     <parent link="table_link"/>
     <child link="support_base_link"/>
-    <origin xyz="0.7 0 0" rpy="0 0 ${pi/2}"/>
+    <origin xyz="0.60 0 0" rpy="0 0 ${pi/2}"/>
   </joint>
   <gazebo>

File: agimus_demo_10_tiago_pro_bar_manip/urdf/macro/table_macro.urdf.xacro (robot description, xacro)
@@ -3,5 +3,5 @@
   <xacro:macro name="table" params="prefix:=''">
     <material name="Blue">
-      <color rgba="0.0 0.05 0.4 1.0"/>
+      <color rgba="0.0 0.0 0.4 1.0"/>
     </material>
     <link name="${prefix}table_link">
@@ -9,17 +9,29 @@
         <origin xyz="0 0 0"/>
         <mass value="25.5"/>
-        <inertia ixx="0.02" ixy="0" ixz="0" iyy="0.05" iyz="0" izz="0.04"/>
+        <inertia ixx="0.02" ixy="0" ixz="0"
+                 iyy="0.05" iyz="0" izz="0.04"/>
       </inertial>
       <visual>
-        <origin rpy="0 0 0" xyz="0 0 -0.05"/>
+        <origin rpy="0 0 0" xyz="0.35 0 0"/>
         <geometry>
-          <mesh filename="package://agimus_demo_10_tiago_pro_bar_manip/meshes/table.stl" scale="0.001 0.001 0.001"/>
+          <mesh
+            filename="package://agimus_demo_10_tiago_pro_bar_manip/meshes/table.stl"
+            scale="0.001 0.001 0.001"/>
+        </geometry>
+        <material name="Blue"/>
+      </visual>
+      <visual>
+        <origin rpy="0 0 0" xyz="-0.35 0 0"/>
+        <geometry>
+          <mesh
+            filename="package://agimus_demo_10_tiago_pro_bar_manip/meshes/table.stl"
+            scale="0.001 0.001 0.001"/>
         </geometry>
         <material name="Blue"/>
       </visual>
       <collision>
-        <origin rpy="0 0 0" xyz="0 0 -0.05"/>
+        <origin rpy="0 0 0" xyz="0 0 -0.37"/>
         <geometry>
-          <mesh filename="package://agimus_demo_10_tiago_pro_bar_manip/meshes/table.stl" scale="0.001 0.001 0.001"/>
+          <box size="1.4 1.4 0.74"/>
         </geometry>
       </collision>

File: agimus_demo_10_tiago_pro_bar_manip/urdf/standalone/table.urdf (robot description, URDF)
Before this commit: robot table, 1 links, 0 joints
Links:
- link table_link: mass None -> 25.5; geometry collision box size=1.4 1.4 0.74; visual mesh filename=package://agimus_demo_10_tiago_pro_bar_manip/meshes/table.s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 scale=0.001 0.001 0.001

File: agimus_demo_10_tiago_pro_bar_manip/urdf/standalone/table.urdf.xacro (robot description, xacro)
@@ -1,14 +1,5 @@
 <?xml version="1.0"?>
-<robot xmlns:xacro="http://www.ros.org/wiki/xacro" name="table">
+<robot name="table" xmlns:xacro="http://www.ros.org/wiki/xacro">
   <xacro:include filename="$(find agimus_demo_10_tiago_pro_bar_manip)/urdf/macro/table_macro.urdf.xacro"/>
-  <link name="world"/>
   <xacro:table prefix=""/>
-  <joint name="world_to_table" type="fixed">
-    <parent link="world"/>
-    <child link="table_link"/>
-    <origin xyz="2. 0 0" rpy="0 0 0"/>
-  </joint>
-  <gazebo>
-    <static>true</static>
-  </gazebo>
 </robot>

Commit message: table link on top of table & plate linked to table and not world

File: agimus_demo_10_tiago_pro_bar_manip/urdf/environment.urdf.xacro (robot description, xacro)
@@ -16,5 +16,5 @@
     <parent link="world"/>
     <child link="table_link"/>
-    <origin xyz="2.9 0 0" rpy="0 0 3.14"/>
+    <origin xyz="2.9 0 0.74" rpy="0 0 3.14"/>
   </joint>
   <xacro:bordered_plate name="plate">
@@ -22,7 +22,7 @@
   </xacro:bordered_plate>
   <joint name="plate_world_joint" type="fixed">
-    <parent link="world"/>
+    <parent link="table_link"/>
     <child link="plate_base_link"/>
-    <origin xyz="2.3 0 0.66" rpy="0 0 0"/>
+    <origin xyz="0 0 0.015" rpy="0 0 0"/>
   </joint>
   <xacro:support_bar spacing="0.95"/>
@@ -30,5 +30,5 @@
     <parent link="table_link"/>
     <child link="support_base_link"/>
-    <origin xyz="1.32 0 0.7" rpy="0 0 ${pi/2}"/>
+    <origin xyz="0.7 0 0" rpy="0 0 ${pi/2}"/>
   </joint>
   <gazebo>

File: agimus_demo_10_tiago_pro_bar_manip/urdf/macro/table_macro.urdf.xacro (robot description, xacro)
@@ -12,5 +12,5 @@
       </inertial>
       <visual>
-        <origin rpy="0 0 0" xyz="0.6 0 0.585"/>
+        <origin rpy="0 0 0" xyz="0 0 -0.05"/>
         <geometry>
           <mesh filename="package://agimus_demo_10_tiago_pro_bar_manip/meshes/table.stl" scale="0.001 0.001 0.001"/>
@@ -19,5 +19,5 @@
       </visual>
       <collision>
-        <origin rpy="0 0 0" xyz="0.6 0 0.585"/>
+        <origin rpy="0 0 0" xyz="0 0 -0.05"/>
         <geometry>
           <mesh filename="package://agimus_demo_10_tiago_pro_bar_manip/meshes/table.stl" scale="0.001 0.001 0.001"/>

Commit message: mocap + unlink table from env

File: agimus_demo_10_tiago_pro_bar_manip/urdf/environment.urdf.xacro (robot description, xacro)
@@ -13,4 +13,5 @@
   </joint>
   <xacro:table/>
+  <!-- <link name="table_link"/> -->
   <joint name="table_world_joint" type="fixed">
     <parent link="world"/>

File: agimus_demo_10_tiago_pro_bar_manip/urdf/standalone/table.urdf.xacro (robot description, xacro)
@@ -1,10 +1,5 @@
-<!-- <?xml version="1.0"?>
-<robot name="table" xmlns:xacro="http://www.ros.org/wiki/xacro">
-  <xacro:include filename="$(find agimus_demo_10_tiago_pro_bar_manip)/urdf/macro/table_macro.urdf.xacro"/>
-  <xacro:table prefix=""/>
-</robot> -->
 <?xml version="1.0"?>
 <robot xmlns:xacro="http://www.ros.org/wiki/xacro" name="table">
-  <xacro:include filename="$(find agimus_demo_10_tiago_pro_bar_manip)/urdf/macro/table_macro.xacro"/>
+  <xacro:include filename="$(find agimus_demo_10_tiago_pro_bar_manip)/urdf/macro/table_macro.urdf.xacro"/>
   <link name="world"/>
   <xacro:table prefix=""/>

Commit message: cleanup launch + tf fix for table mocap

File: agimus_demo_10_tiago_pro_bar_manip/urdf/environment.urdf.xacro (robot description, xacro)
@@ -16,5 +16,5 @@
   <joint name="table_world_joint" type="fixed">
     <parent link="world"/>
-    <child link="table_link"/>
+    <child link="mocap_table"/>
     <origin xyz="2.3 0 0.74" rpy="0 0 3.14"/>
   </joint>

File: agimus_demo_10_tiago_pro_bar_manip/urdf/macro/table_macro.urdf.xacro (robot description, xacro)
@@ -5,4 +5,10 @@
       <color rgba="0.0 0.0 0.4 1.0"/>
     </material>
+    <link name="mocap_table"/>
+    <joint name="mocap_to_table" type="fixed">
+      <parent link="mocap_table"/>
+      <child link="table_link"/>
+      <origin xyz="0.7 -0.7 0" rpy="0 0 1.57"/>
+    </joint>
     <link name="${prefix}table_link">
       <inertial>
@@ -37,10 +43,4 @@
       </collision>
     </link>
-    <link name="mocap_table"/>
-    <joint name="mocap_to_table" type="fixed">
-      <parent link="table_link"/>
-      <child link="mocap_table"/>
-      <origin xyz="0.7 -0.7 0" rpy="0 0 1.57"/>
-    </joint>
   </xacro:macro>
 </robot>

Commit message: adjustements bar placement & link mocap for table

File: agimus_demo_10_tiago_pro_bar_manip/urdf/environment.urdf.xacro (robot description, xacro)
@@ -16,6 +16,6 @@
   <joint name="table_world_joint" type="fixed">
     <parent link="world"/>
-    <child link="mocap_table"/>
-    <origin xyz="2.3 0 0.74" rpy="0 0 3.14"/>
+    <child link="table_mocap"/>
+    <origin xyz="2 0.7 0.74" rpy="0 0 -${pi/2}"/>
   </joint>
   <xacro:bordered_plate name="plate">

File: agimus_demo_10_tiago_pro_bar_manip/urdf/macro/table_macro.urdf.xacro (robot description, xacro)
@@ -5,9 +5,9 @@
       <color rgba="0.0 0.0 0.4 1.0"/>
     </material>
-    <link name="mocap_table"/>
+    <link name="table_mocap"/>
     <joint name="mocap_to_table" type="fixed">
-      <parent link="mocap_table"/>
+      <parent link="table_mocap"/>
       <child link="table_link"/>
-      <origin xyz="0.7 -0.7 0" rpy="0 0 1.57"/>
+      <origin xyz="0.7 0.7 0" rpy="0 0 -${pi/2}"/>
     </joint>
     <link name="${prefix}table_link">
